File: christmas-tree.kicad_pcb (KiCad board)
At the start: 2 copper layers, 75 x 100 mm, 16 parts, among them U1 PY32F002AL15S6TU

Commit message: JLC Order placed #1
Routing:
- net Net-(D1-K): track 97.0 -> 105.6 mm
- net GND: vias 1 -> 5
