File: christmas-tree.kicad_sch (KiCad schematic)
At the start: 16 parts, among them U1 PY32F002AL15S6TU

Commit message: JLC Order placed #1
Parts:
- BT1: footprint Battery:BatteryHolder_Keystone_3002_1x2032 -> OneOffs:BatteryHolder_WJ-CR2032-1-W
- R1, R2, R3, R4: value 120 -> 33
Changed lines of the file:
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@@
 			)
 		)
-		(property "Value" "120"
+		(property "Value" "33"
 			(at 144.78 111.76 90)
 			(effects
@@
 			)
 		)
-		(property "Value" "120"
+		(property "Value" "33"
 			(at 129.54 114.3 90)
 			(effects
@@
 			)
 		)
-		(property "Footprint" "Battery:BatteryHolder_Keystone_3002_1x2032"
+		(property "Footprint" "OneOffs:BatteryHolder_WJ-CR2032-1-W"
 			(at 199.39 148.336 90)
 			(effects
@@
 			)
 		)
-		(property "Value" "120"
+		(property "Value" "33"
 			(at 160.02 109.22 90)
 			(effects
@@
 			)
 		)
-		(property "Value" "120"
+		(property "Value" "33"
 			(at 175.26 106.68 90)
 			(effects
